File: compatible-chan-v0-led/compatible_chan-v0-led.kicad_sch (KiCad schematic)
At the start: 11 parts, among them J1 Conn_01x07_Pin, U1 MAX7219, U2 MAX7219

Commit message: LED版関連更新 基板更新,シェル設計
Parts:
- added C1, C2: 100n, Capacitor_SMD:C_0805_2012Metric_Pad1.18x1.45mm_HandSolder, symbol Device:C
- added C3, C4: 10u, Capacitor_Tantalum_SMD:CP_EIA-2012-15_AVX-P_Pad1.30x1.05mm_HandSolder, symbol Device:C_Polarized
- added J2: SERVO1, Connector_PinHeader_2.54mm:PinHeader_1x03_P2.54mm_Vertical, symbol Connector:Conn_01x03_Pin
- added J3: SERVO2, Connector_PinHeader_2.54mm:PinHeader_1x03_P2.54mm_Vertical, symbol Connector:Conn_01x03_Pin
- J1: value Conn_01x07_Pin -> EXT
Connections:
- net DIN: now also J1.3 (Pin_3); no longer J1.5 (Pin_5)
- net GND: now also J1.6 (Pin_6), C1.2, C2.2, C3.2, C4.2, J2.3 (Pin_3), J3.3 (Pin_3); no longer J1.2 (Pin_2)
- net LOAD: now also J1.5 (Pin_5); no longer J1.3 (Pin_3)
- net SIG1: now also J1.2 (Pin_2), J2.1 (Pin_1); no longer J1.6 (Pin_6)
- net SIG2: now also J1.1 (Pin_1), J3.1 (Pin_1); no longer J1.7 (Pin_7)
- net VCC: now also J1.7 (Pin_7), C1.1, C2.1, C3.1, C4.1, J2.2 (Pin_2), J3.2 (Pin_2); no longer J1.1 (Pin_1)

Commit message: v0-led基板更新、テストファーム・v0.1用MCU基板追加
Parts:
- D1, D2: value 788AS -> 788BS
Connections:
- net D1.0: now also D1.13 (C1); no longer D1.9 (R1)
- net D1.1: now also D1.3 (C2); no longer D1.14 (R2)
- net D1.2: now also D1.4 (C3); no longer D1.8 (R3)
- net D1.3: now also D1.10 (C4); no longer D1.12 (R4)
- net D1.4: now also D1.6 (C5); no longer D1.1 (R5)
- net D1.5: now also D1.11 (C6); no longer D1.7 (R6)
- net D1.6: now also D1.15 (C7); no longer D1.2 (R7)
- net D1.7: now also D1.16 (C8); no longer D1.5 (R8)
- net D1.A: now also D1.2 (R7); no longer D1.3 (C2)
- net D1.B: now also D1.7 (R6); no longer D1.4 (C3)
- net D1.C: now also D1.1 (R5); no longer D1.10 (C4)
- net D1.D: now also D1.12 (R4); no longer D1.6 (C5)
- net D1.DP: now also D1.5 (R8); no longer D1.13 (C1)
- net D1.E: now also D1.8 (R3); no longer D1.11 (C6)
- net D1.F: now also D1.14 (R2); no longer D1.15 (C7)
- net D1.G: now also D1.9 (R1); no longer D1.16 (C8)
- net D2.0: now also D2.13 (C1); no longer D2.9 (R1)
- net D2.1: now also D2.3 (C2); no longer D2.14 (R2)
- net D2.2: now also D2.4 (C3); no longer D2.8 (R3)
- net D2.3: now also D2.10 (C4); no longer D2.12 (R4)
- net D2.4: now also D2.6 (C5); no longer D2.1 (R5)
- net D2.5: now also D2.11 (C6); no longer D2.7 (R6)
- net D2.6: now also D2.15 (C7); no longer D2.2 (R7)
- net D2.7: now also D2.16 (C8); no longer D2.5 (R8)
- net D2.A: now also D2.2 (R7); no longer D2.3 (C2)
- net D2.B: now also D2.7 (R6); no longer D2.4 (C3)
- net D2.C: now also D2.1 (R5); no longer D2.10 (C4)
- net D2.D: now also D2.12 (R4); no longer D2.6 (C5)
- net D2.DP: now also D2.5 (R8); no longer D2.13 (C1)
- net D2.E: now also D2.8 (R3); no longer D2.11 (C6)
- net D2.F: now also D2.14 (R2); no longer D2.15 (C7)
- net D2.G: now also D2.9 (R1); no longer D2.16 (C8)
Changed lines of the file:
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@@
 		)
 	)
-	(label "D1.1"
+	(label "D1.F"
 		(at 78.7438 120.65 0)
 		(fields_autoplaced yes)
@@
 		)
 	)
-	(label "D1.F"
+	(label "D1.6"
 		(at 119.3762 133.35 0)
 		(fields_autoplaced yes)
@@
 		)
 	)
-	(label "D1.E"
+	(label "D1.5"
 		(at 119.38 130.81 0)
 		(fields_autoplaced yes)
@@
 		)
 	)
-	(label "D2.D"
+	(label "D2.4"
 		(at 241.3038 128.27 0)
 		(fields_autoplaced yes)
@@
 		)
 	)
-	(label "D1.C"
+	(label "D1.3"
 		(at 119.38 125.73 0)
 		(fields_autoplaced yes)
@@
 		)
 	)
-	(label "D1.A"
+	(label "D1.1"
 		(at 119.38 120.65 0)
 		(fields_autoplaced yes)
@@
 		)
 	)
-	(label "D2.B"
+	(label "D2.2"
 		(at 241.3038 123.19 0)
 		(fields_autoplaced yes)
@@
 		)
 	)
-	(label "D1.6"
+	(label "D1.A"
 		(at 78.7438 133.35 0)
 		(fields_autoplaced yes)
@@
 		)
 	)
-	(label "D2.7"
+	(label "D2.DP"
 		(at 200.6638 135.89 0)
 		(fields_autoplaced yes)
@@
 		)
 	)
-	(label "D1.D"
+	(label "D1.4"
 		(at 119.38 128.27 0)
 		(fields_autoplaced yes)
@@
 		)
 	)
-	(label "D2.DP"
+	(label "D2.0"
 		(at 241.3 118.11 0)
 		(fields_autoplaced yes)
@@
 		)
 	)
-	(label "D1.5"
+	(label "D1.B"
 		(at 78.74 130.81 0)
 		(fields_autoplaced yes)
@@
 		)
 	)
-	(label "D1.3"
+	(label "D1.D"
 		(at 78.74 125.73 0)
 		(fields_autoplaced yes)
@@
 		)
 	)
-	(label "D1.DP"
+	(label "D1.0"
 		(at 119.38 118.11 0)
 		(fields_autoplaced yes)
@@
 		)
 	)
-	(label "D1.B"
+	(label "D1.2"
 		(at 119.38 123.19 0)
 		(fields_autoplaced yes)
@@
 		)
 	)
-	(label "D2.0"
+	(label "D2.G"
 		(at 200.6638 118.11 0)
 		(fields_autoplaced yes)
@@
 		)
 	)
-	(label "D1.4"
+	(label "D1.C"
 		(at 78.7438 128.27 0)
 		(fields_autoplaced yes)
@@
 		)
 	)
-	(label "D2.4"
+	(label "D2.C"
 		(at 200.6638 128.27 0)
 		(fields_autoplaced yes)
@@
 		)
 	)
-	(label "D2.E"
+	(label "D2.5"
 		(at 241.3038 130.81 0)
 		(fields_autoplaced yes)
@@
 		)
 	)
-	(label "D2.G"
+	(label "D2.7"
 		(at 241.3038 135.89 0)
 		(fields_autoplaced yes)
@@
 		)
 	)
-	(label "D1.2"
+	(label "D1.E"
 		(at 78.7438 123.19 0)
 		(fields_autoplaced yes)
@@
 		)
 	)
-	(label "D2.6"
+	(label "D2.A"
 		(at 200.6638 133.35 0)
 		(fields_autoplaced yes)
@@
 		)
 	)
-	(label "D2.C"
+	(label "D2.3"
 		(at 241.3038 125.73 0)
 		(fields_autoplaced yes)
@@
 		)
 	)
-	(label "D1.7"
+	(label "D1.DP"
 		(at 78.7438 135.89 0)
 		(fields_autoplaced yes)
@@
 		)
 	)
-	(label "D2.2"
+	(label "D2.E"
 		(at 200.6638 123.19 0)
 		(fields_autoplaced yes)
@@
 		)
 	)
-	(label "D1.0"
+	(label "D1.G"
 		(at 78.7438 118.11 0)
 		(fields_autoplaced yes)
@@
 		)
 	)
-	(label "D2.1"
+	(label "D2.F"
 		(at 200.6638 120.65 0)
 		(fields_autoplaced yes)
@@
 		)
 	)
-	(label "D2.5"
+	(label "D2.B"
 		(at 200.66 130.81 0)
 		(fields_autoplaced yes)
@@
 		)
 	)
-	(label "D1.G"
+	(label "D1.7"
 		(at 119.38 135.89 0)
 		(fields_autoplaced yes)
@@
 		)
 	)
-	(label "D2.A"
+	(label "D2.1"
 		(at 241.3038 120.65 0)
 		(fields_autoplaced yes)
@@
 		)
 	)
-	(label "D2.3"
+	(label "D2.D"
 		(at 200.66 125.73 0)
 		(fields_autoplaced yes)
@@
 		)
 	)
-	(label "D2.F"
+	(label "D2.6"
 		(at 241.3 133.35 0)
 		(fields_autoplaced yes)
@@
 			)
 		)
-		(property "Value" "788AS"
+		(property "Value" "788BS"
 			(at 100.965 113.03 0)
 			(effects
@@
 			)
 		)
-		(property "Value" "788AS"
+		(property "Value" "788BS"
 			(at 222.885 113.03 0)
 			(effects
